File: lab4/555_Timer_Based_Circuit/555_Timer_Based_Circuit.kicad_sch (KiCad schematic)
At the start: 10 parts, among them J1 J1, U1 NE555D

Commit message: Add files via upload
Parts:
- C1: footprint (none) -> C_0805_2012Metric_Pad1.18x1.45mm_HandSolder
- C2: footprint (none) -> CP_EIA-3216-18_Kemet-A_Pad1.58x1.35mm_HandSolder
- D1, D2: footprint (none) -> LED_1206_3216Metric_Pad1.42x1.75mm_HandSolder
- J1: footprint (none) -> TerminalBlock_bornier-2_P5.08mm
- R1, R2, R3, R4: footprint (none) -> R_0805_2012Metric_Pad1.20x1.40mm_HandSolder
- U1: footprint Package_SO:SOIC-8_3.9x4.9mm_P1.27mm -> SOIC-8-1EP_3.9x4.9mm_P1.27mm_EP2.29x3mm
Changed lines of the file:
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@@
       (effects (font (size 1.27 1.27)) (justify left) hide)
     )
-    (property "Footprint" "Package_SO:SOIC-8_3.9x4.9mm_P1.27mm" (id 2) (at 167.64 115.57 0)
+    (property "Footprint" "SOIC-8-1EP_3.9x4.9mm_P1.27mm_EP2.29x3mm" (id 2) (at 167.64 115.57 0)
       (effects (font (size 1.27 1.27)) hide)
     )
@@
       (effects (font (size 1.27 1.27)) (justify left))
     )
-    (property "Footprint" "" (id 2) (at 183.642 113.03 90)
+    (property "Footprint" "R_0805_2012Metric_Pad1.20x1.40mm_HandSolder" (id 2) (at 183.642 113.03 90)
       (effects (font (size 1.27 1.27)) hide)
     )
@@
       (effects (font (size 1.27 1.27)) (justify left))
     )
-    (property "Footprint" "" (id 2) (at 183.642 97.79 90)
+    (property "Footprint" "R_0805_2012Metric_Pad1.20x1.40mm_HandSolder" (id 2) (at 183.642 97.79 90)
       (effects (font (size 1.27 1.27)) hide)
     )
@@
       (effects (font (size 1.27 1.27)) (justify left))
     )
-    (property "Footprint" "" (id 2) (at 115.2652 128.27 0)
+    (property "Footprint" "C_0805_2012Metric_Pad1.18x1.45mm_HandSolder" (id 2) (at 115.2652 128.27 0)
       (effects (font (size 1.27 1.27)) hide)
     )
@@
       (effects (font (size 1.27 1.27)) (justify left))
     )
-    (property "Footprint" "" (id 2) (at 84.582 85.09 90)
+    (property "Footprint" "R_0805_2012Metric_Pad1.20x1.40mm_HandSolder" (id 2) (at 84.582 85.09 90)
       (effects (font (size 1.27 1.27)) hide)
     )
@@
       (effects (font (size 1.27 1.27)) (justify left))
     )
-    (property "Footprint" "" (id 2) (at 87.3252 130.81 0)
+    (property "Footprint" "CP_EIA-3216-18_Kemet-A_Pad1.58x1.35mm_HandSolder" (id 2) (at 87.3252 130.81 0)
       (effects (font (size 1.27 1.27)) hide)
     )
@@
       (effects (font (size 1.27 1.27)) (justify left))
     )
-    (property "Footprint" "" (id 2) (at 84.582 107.95 90)
+    (property "Footprint" "R_0805_2012Metric_Pad1.20x1.40mm_HandSolder" (id 2) (at 84.582 107.95 90)
       (effects (font (size 1.27 1.27)) hide)
     )
@@
       (effects (font (size 1.27 1.27)) (justify right))
     )
-    (property "Footprint" "" (id 2) (at 185.42 129.54 0)
+    (property "Footprint" "LED_1206_3216Metric_Pad1.42x1.75mm_HandSolder" (id 2) (at 185.42 129.54 0)
       (effects (font (size 1.27 1.27)) hide)
     )
@@
       (effects (font (size 1.27 1.27)) (justify right))
     )
-    (property "Footprint" "" (id 2) (at 185.42 83.82 0)
+    (property "Footprint" "LED_1206_3216Metric_Pad1.42x1.75mm_HandSolder" (id 2) (at 185.42 83.82 0)
       (effects (font (size 1.27 1.27)) hide)
     )
@@
     )
     (property "Value" "J1" (id 1) (at 143.51 73.66 0))
-    (property "Footprint" "" (id 2) (at 138.43 73.66 0)
+    (property "Footprint" "TerminalBlock_bornier-2_P5.08mm" (id 2) (at 138.43 73.66 0)
       (effects (font (size 1.27 1.27)) hide)
     )
@@
   (symbol (lib_id "power:+9V") (at 146.05 86.36 0) (unit 1)
     (in_bom yes) (on_board yes) (fields_autoplaced)
-    (property "Reference" "#PWR?" (id 0) (at 146.05 90.17 0)
+    (property "Reference" "#PWR0101" (id 0) (at 146.05 90.17 0)
       (effects (font (size 1.27 1.27)) hide)
     )
@@
     )
     (path "/f5fc9f09-c386-4372-a072-e9cbb94b8cd5"
-      (reference "#PWR?") (unit 1) (value "+9V") (footprint "")
+      (reference "#PWR0101") (unit 1) (value "+9V") (footprint "")
     )
     (path "/23465697-ba48-4b36-9028-37a63bae271b"
-      (reference "C1") (unit 1) (value "0.01 μF") (footprint "")
+      (reference "C1") (unit 1) (value "0.01 μF") (footprint "C_0805_2012Metric_Pad1.18x1.45mm_HandSolder")
     )
     (path "/5bef235e-c5be-4302-ac5b-2a6326b27402"
-      (reference "C2") (unit 1) (value "10 μF") (footprint "")
+      (reference "C2") (unit 1) (value "10 μF") (footprint "CP_EIA-3216-18_Kemet-A_Pad1.58x1.35mm_HandSolder")
     )
     (path "/e1e4d2fc-4e94-48a1-afaa-30b7077b92e0"
-      (reference "D1") (unit 1) (value "LED") (footprint "")
+      (reference "D1") (unit 1) (value "LED") (footprint "LED_1206_3216Metric_Pad1.42x1.75mm_HandSolder")
     )
     (path "/cfde45f3-6407-4204-85b5-e5fcf2dbf58a"
-      (reference "D2") (unit 1) (value "LED") (footprint "")
+      (reference "D2") (unit 1) (value "LED") (footprint "LED_1206_3216Metric_Pad1.42x1.75mm_HandSolder")
     )
     (path "/f259d4c5-41e1-4e9d-b856-7940fb6948de"
-      (reference "J1") (unit 1) (value "J1") (footprint "")
+      (reference "J1") (unit 1) (value "J1") (footprint "TerminalBlock_bornier-2_P5.08mm")
     )
     (path "/49a2ba63-d010-41ef-be76-d27c72185c0d"
-      (reference "R1") (unit 1) (value "1k") (footprint "")
+      (reference "R1") (unit 1) (value "1k") (footprint "R_0805_2012Metric_Pad1.20x1.40mm_HandSolder")
     )
     (path "/22d59abf-d2ee-48cf-b1b6-76f2383b68a7"
-      (reference "R2") (unit 1) (value "1k") (footprint "")
+      (reference "R2") (unit 1) (value "1k") (footprint "R_0805_2012Metric_Pad1.20x1.40mm_HandSolder")
     )
     (path "/67c31c46-99c2-43f4-bf1a-50327fd8380d"
-      (reference "R3") (unit 1) (value "10k") (footprint "")
+      (reference "R3") (unit 1) (value "10k") (footprint "R_0805_2012Metric_Pad1.20x1.40mm_HandSolder")
     )
     (path "/15ccb520-14c0-4d25-84d0-891a17b54dbd"
-      (reference "R4") (unit 1) (value "1k") (footprint "")
+      (reference "R4") (unit 1) (value "1k") (footprint "R_0805_2012Metric_Pad1.20x1.40mm_HandSolder")
     )
     (path "/1543a055-0a89-4f59-8112-244de6d3ba82"
-      (reference "U1") (unit 1) (value "NE555D") (footprint "Package_SO:SOIC-8_3.9x4.9mm_P1.27mm")
-    )
-  )
+      (reference "U1") (unit 1) (value "NE555D") (footprint "SOIC-8-1EP_3.9x4.9mm_P1.27mm_EP2.29x3mm")
+    )
+  )
