File: lab4/LED_Switch_Circuit/LED_Switch_Circuit.kicad_sch (KiCad schematic)
At the start: 6 parts, among them SW1 SW_SPDT

Commit message: Add files via upload
Parts:
- C1: footprint (none) -> C_Radial_D5.0mm_H5.0mm_P2.00mm
- D1: footprint (none) -> LED_D5.0mm
- R1, R2: footprint (none) -> R_Axial_DIN0516_L15.5mm_D5.0mm_P20.32mm_Horizontal
- SW1: footprint (none) -> SW_E-Switch_EG1224_SPDT_Angled
- V1: footprint (none) -> JST_PH_B2B-PH-K_1x02_P2.00mm_Vertical
Changed lines of the file:
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@@
       (effects (font (size 1.27 1.27)) (justify left))
     )
-    (property "Footprint" "" (id 2) (at 173.6852 95.25 0)
+    (property "Footprint" "C_Radial_D5.0mm_H5.0mm_P2.00mm" (id 2) (at 173.6852 95.25 0)
       (effects (font (size 1.27 1.27)) hide)
     )
@@
       (effects (font (size 1.27 1.27)) (justify left))
     )
-    (property "Footprint" "" (id 2) (at 191.262 82.55 90)
+    (property "Footprint" "R_Axial_DIN0516_L15.5mm_D5.0mm_P20.32mm_Horizontal" (id 2) (at 191.262 82.55 90)
       (effects (font (size 1.27 1.27)) hide)
     )
@@
       (effects (font (size 1.27 1.27)) (justify right) hide)
     )
-    (property "Footprint" "" (id 2) (at 193.04 99.06 0)
+    (property "Footprint" "LED_D5.0mm" (id 2) (at 193.04 99.06 0)
       (effects (font (size 1.27 1.27)) hide)
     )
@@
       (effects (font (size 1.27 1.27)) hide)
     )
-    (property "Footprint" "" (id 2) (at 160.02 76.2 0)
+    (property "Footprint" "SW_E-Switch_EG1224_SPDT_Angled" (id 2) (at 160.02 76.2 0)
       (effects (font (size 1.27 1.27)) hide)
     )
@@
     (property "Reference" "V1" (id 0) (at 132.715 83.82 0))
     (property "Value" "9 V" (id 1) (at 132.715 86.36 0))
-    (property "Footprint" "" (id 2) (at 132.08 88.9 0)
+    (property "Footprint" "JST_PH_B2B-PH-K_1x02_P2.00mm_Vertical" (id 2) (at 132.08 88.9 0)
       (effects (font (size 1.27 1.27)) hide)
     )
@@
     (property "Reference" "R1" (id 0) (at 143.51 69.85 90))
     (property "Value" "2.2 kΩ" (id 1) (at 143.51 72.39 90))
-    (property "Footprint" "" (id 2) (at 143.51 74.422 90)
+    (property "Footprint" "R_Axial_DIN0516_L15.5mm_D5.0mm_P20.32mm_Horizontal" (id 2) (at 143.51 74.422 90)
       (effects (font (size 1.27 1.27)) hide)
     )
@@
   (symbol_instances
     (path "/044e40cb-d22c-43f1-b5f0-025dcda1771b"
-      (reference "C1") (unit 1) (value "4.7 μF") (footprint "")
+      (reference "C1") (unit 1) (value "4.7 μF") (footprint "C_Radial_D5.0mm_H5.0mm_P2.00mm")
     )
     (path "/5e2c1259-0a91-48a8-ae71-817c1341d2f5"
-      (reference "D1") (unit 1) (value "LED") (footprint "")
+      (reference "D1") (unit 1) (value "LED") (footprint "LED_D5.0mm")
     )
     (path "/fa6be15e-086d-442d-b054-fd839d6bc9b2"
-      (reference "R1") (unit 1) (value "2.2 kΩ") (footprint "")
+      (reference "R1") (unit 1) (value "2.2 kΩ") (footprint "R_Axial_DIN0516_L15.5mm_D5.0mm_P20.32mm_Horizontal")
     )
     (path "/43f586c9-5c50-4e37-81a4-0fba01f4e2f3"
-      (reference "R2") (unit 1) (value "20 kΩ") (footprint "")
+      (reference "R2") (unit 1) (value "20 kΩ") (footprint "R_Axial_DIN0516_L15.5mm_D5.0mm_P20.32mm_Horizontal")
     )
     (path "/be40a689-7e7d-4ca8-a7fa-7062c7440650"
-      (reference "SW1") (unit 1) (value "SW_SPDT") (footprint "")
+      (reference "SW1") (unit 1) (value "SW_SPDT") (footprint "SW_E-Switch_EG1224_SPDT_Angled")
     )
     (path "/c45512f9-7e83-481d-9856-ecf0244cd21e"
-      (reference "V1") (unit 1) (value "9 V") (footprint "")
+      (reference "V1") (unit 1) (value "9 V") (footprint "JST_PH_B2B-PH-K_1x02_P2.00mm_Vertical")
     )
   )
